Commit message: ok wrting better top down parcel (wip)

File: newton-4.00/applications/media/r2d3.urdf (robot description, URDF)
Before this commit: robot physics, 2 links, 1 joints
Links:
- added link right_base, mass 10; collision box size=0.4 0.1 0.1; visual box size=0.4 0.1 0.1
Joints:
- added joint right_base_joint: type fixed, parent right_leg, child right_base, origin xyz=0 0 -0.6

Commit message: more urdf parcel (wip)

File: newton-4.00/applications/media/r2d3.urdf (robot description, URDF)
Before this commit: robot physics, 3 links, 2 joints
Links:
- added link right_back_wheel, mass 1; collision cylinder length=0.1 radius=0.035; visual cylinder length=0.1 radius=0.035
- added link right_front_wheel, mass 1; collision cylinder length=0.1 radius=0.035; visual cylinder length=0.1 radius=0.035
Joints:
- added joint right_back_wheel_joint: type continuous, parent right_base, child right_back_wheel, origin xyz=-0.133333333333 0 -0.085 rpy=0 0 0, axis 0 1 0
- added joint right_front_wheel_joint: type continuous, parent right_base, child right_front_wheel, origin xyz=0.133333333333 0 -0.085 rpy=0 0 0, axis 0 1 0
