Commit message: debugging urdf exporter (wip)

File: newton-4.00/applications/media/r2d2__.urdf (robot description, URDF)
Before this commit: robot physics, 2 links, 1 joints
Links:
- removed link right_leg
- added link head, mass 2; collision sphere radius=0.2; visual sphere radius=0.2
Joints:
- removed joint base_to_right_leg
- added joint head_swivel: type continuous, parent base_link, child head, origin xyz=0 0 0.3, axis 0 0 1
