Commit message: improve urdf files import/export funtionality. nwo test with more complex models.

File: newton-4.00/applications/media/cartpoleHandMade.urdf (robot description, URDF)
Before this commit: robot robot_model, 2 links, 1 joints
Joints:
- joint node_0_link_to_base_link: origin xyz=0 1.96198e-08 0.0625 rpy=3.13916e-07 -0 1.5708 -> xyz=0 0 0 rpy=0 0 1.57075

File: newton-4.00/applications/media/unicycle.urdf (robot description, URDF)
Before this commit: robot robot_model, 3 links, 2 joints
Joints:
- joint node_0_link_to_node_1_link: axis 3.13916e-07 -1 3.13916e-07 -> (none); origin xyz=-0.3 0 0 rpy=6.27833e-07 -1.5708 0 -> xyz=-4.52987e-08 -4.52987e-08 0.3 rpy=0 -0 -1.68775e-21
- joint node_1_link_to_base_link: axis 3.13916e-07 -1 3.13916e-07 -> (none); origin xyz=0 -6.27833e-08 -0.2 rpy=6.27833e-07 -1.5708 0 -> xyz=0 -3.01992e-08 -0.2 rpy=3.14159 -3.01992e-07 -1.5708
