Commit message: playing trained quad spider walk.

File: newton-4.00/applications/media/quadSpider.urdf (robot description, URDF)
Before this commit: robot robot_model, 13 links, 12 joints
Links:
- removed link node_0_link
- removed link node_10_link
- removed link node_11_link
- removed link node_1_link
- removed link node_2_link
- removed link node_3_link
- removed link node_4_link
- removed link node_5_link
- removed link node_6_link
- removed link node_7_link
- removed link node_8_link
- removed link node_9_link
- added link calf_0, mass 0.0625; collision cylinder length=0.4 radius=0.05; visual cylinder length=0.4 radius=0.05
- added link calf_1, mass 0.0625; collision cylinder length=0.4 radius=0.05; visual cylinder length=0.4 radius=0.05
- added link calf_2, mass 0.0625; collision cylinder length=0.4 radius=0.05; visual cylinder length=0.4 radius=0.05
- added link calf_3, mass 0.0625; collision cylinder length=0.4 radius=0.05; visual cylinder length=0.4 radius=0.05
- added link foot_0, mass 0.0625; collision cylinder length=0.25 radius=0.05; visual cylinder length=0.25 radius=0.05
- added link foot_1, mass 0.0625; collision cylinder length=0.25 radius=0.05; visual cylinder length=0.25 radius=0.05
- added link foot_2, mass 0.0625; collision cylinder length=0.25 radius=0.05; visual cylinder length=0.25 radius=0.05
- added link foot_3, mass 0.0625; collision cylinder length=0.25 radius=0.05; visual cylinder length=0.25 radius=0.05
- added link thigh_0, mass 0.25; collision cylinder length=0.4 radius=0.05; visual cylinder length=0.4 radius=0.05
- added link thigh_1, mass 0.25; collision cylinder length=0.4 radius=0.05; visual cylinder length=0.4 radius=0.05
- added link thigh_2, mass 0.25; collision cylinder length=0.4 radius=0.05; visual cylinder length=0.4 radius=0.05
- added link thigh_3, mass 0.25; collision cylinder length=0.4 radius=0.05; visual cylinder length=0.4 radius=0.05
Joints:
- removed joint node_0_link_to_node_1_link
- removed joint node_10_link_to_node_11_link
- removed joint node_11_link_to_base_link
- removed joint node_1_link_to_node_2_link
- removed joint node_2_link_to_base_link
- removed joint node_3_link_to_node_4_link
- removed joint node_4_link_to_node_5_link
- removed joint node_5_link_to_base_link
- removed joint node_6_link_to_node_7_link
- removed joint node_7_link_to_node_8_link
- removed joint node_8_link_to_base_link
- removed joint node_9_link_to_node_10_link
- added joint calf_0_to_thigh_0: type floating, parent thigh_0, child calf_0, origin xyz=0.3 0 -2.63088e-08 rpy=3.14159 1.5708 0
- added joint calf_1_to_thigh_1: type floating, parent thigh_1, child calf_1, origin xyz=0.3 1.49012e-08 8.42733e-09 rpy=3.14159 1.5708 0
- added joint calf_2_to_thigh_2: type floating, parent thigh_2, child calf_2, origin xyz=0.3 2.98023e-08 -3.49351e-09 rpy=-3.14159 -1.5708 0
- added joint calf_3_to_thigh_3: type floating, parent thigh_3, child calf_3, origin xyz=0.3 0 5.13314e-10 rpy=-3.14159 -1.5708 0
- added joint foot_0_to_calf_0: type continuous, parent calf_0, child foot_0, origin xyz=3.49347e-09 0.3 -2.98023e-08 rpy=-0.785398 -8.22321e-09 3.14159
- added joint foot_1_to_calf_1: type continuous, parent calf_1, child foot_1, origin xyz=-5.26674e-08 0.3 -5.96046e-08 rpy=-0.785398 -6.67831e-09 3.14159
- added joint foot_2_to_calf_2: type continuous, parent calf_2, child foot_2, origin xyz=-5.01507e-08 0.3 -2.98023e-08 rpy=2.35619 -6.78278e-08 -9.76301e-08
- added joint foot_3_to_calf_3: type continuous, parent calf_3, child foot_3, origin xyz=1.58779e-08 0.3 -5.96046e-08 rpy=2.35619 8.27288e-08 2.31242e-08
- added joint thigh_0_to_base_link: type floating, parent base_link, child thigh_0, origin xyz=0.1125 -0.194856 -0.125 rpy=1.5708 -0.785398 -1.0472
- added joint thigh_1_to_base_link: type floating, parent base_link, child thigh_1, origin xyz=-0.1125 -0.194856 -0.125 rpy=1.5708 -0.785398 -2.0944
- added joint thigh_2_to_base_link: type floating, parent base_link, child thigh_2, origin xyz=-0.1125 0.194856 -0.125 rpy=1.5708 -0.785398 2.09439
- added joint thigh_3_to_base_link: type floating, parent base_link, child thigh_3, origin xyz=0.1125 0.194856 -0.125 rpy=1.5708 -0.785398 1.0472

Commit message: some wrdf fixes

File: newton-4.00/applications/media/quadSpider.urdf (robot description, URDF)
Before this commit: robot robot_model, 13 links, 12 joints
Joints:
- joint calf_0_to_thigh_0: limit (none) -> lower=-1.221730 upper=1.221730 effort=1000.000000 velocity=0.500000; type floating -> revolute
- joint calf_1_to_thigh_1: limit (none) -> lower=-1.221730 upper=1.221730 effort=1000.000000 velocity=0.500000; type floating -> revolute
- joint calf_2_to_thigh_2: limit (none) -> lower=-1.221730 upper=1.221730 effort=1000.000000 velocity=0.500000; type floating -> revolute
- joint calf_3_to_thigh_3: limit (none) -> lower=-1.221730 upper=1.221730 effort=1000.000000 velocity=0.500000; type floating -> revolute

Commit message: tuning pose matching trainier
still lots of problems

File: newton-4.00/applications/media/quadSpider.urdf (robot description, URDF)
Before this commit: robot robot_model, 13 links, 12 joints
Joints:
- joint calf_0_to_thigh_0: limit lower=-1.221730 upper=1.221730 effort=1000.000000 velocity=0.500000 -> lower=-1.047197 upper=1.047197 effort=1000.000000 velocity=0.500000; origin xyz=0.3 0 -2.63088e-08 rpy=3.14159 1.5708 0 -> xyz=0.3 -5.55112e-17 2.39534e-17 rpy=3.14159 1.5708 0
- joint calf_1_to_thigh_1: limit lower=-1.221730 upper=1.221730 effort=1000.000000 velocity=0.500000 -> lower=-1.047197 upper=1.047197 effort=1000.000000 velocity=0.500000; origin xyz=0.3 1.49012e-08 8.42733e-09 rpy=3.14159 1.5708 0 -> xyz=0.3 1.11022e-16 5.07754e-17 rpy=3.14159 1.5708 0
- joint calf_2_to_thigh_2: limit lower=-1.221730 upper=1.221730 effort=1000.000000 velocity=0.500000 -> lower=-1.047197 upper=1.047197 effort=1000.000000 velocity=0.500000; origin xyz=0.3 2.98023e-08 -3.49351e-09 rpy=-3.14159 -1.5708 0 -> xyz=0.3 2.77556e-17 2.45631e-17 rpy=-3.14159 -1.5708 0
- joint calf_3_to_thigh_3: limit lower=-1.221730 upper=1.221730 effort=1000.000000 velocity=0.500000 -> lower=-1.047197 upper=1.047197 effort=1000.000000 velocity=0.500000; origin xyz=0.3 0 5.13314e-10 rpy=-3.14159 -1.5708 0 -> xyz=0.3 -2.77556e-17 -2.45058e-17 rpy=-3.14159 -1.5708 0
- joint foot_0_to_calf_0: origin xyz=3.49347e-09 0.3 -2.98023e-08 rpy=-0.785398 -8.22321e-09 3.14159 -> xyz=3.08777e-17 0.3 -5.55112e-17 rpy=-0.785398 -4.88977e-17 -3.14159
- joint foot_1_to_calf_1: origin xyz=-5.26674e-08 0.3 -5.96046e-08 rpy=-0.785398 -6.67831e-09 3.14159 -> xyz=-2.54984e-17 0.3 -5.55112e-17 rpy=-0.785398 4.80945e-17 3.14159
- joint foot_2_to_calf_2: origin xyz=-5.01507e-08 0.3 -2.98023e-08 rpy=2.35619 -6.78278e-08 -9.76301e-08 -> xyz=-7.58832e-17 0.3 -5.55112e-17 rpy=2.35619 -4.40315e-17 -1.85238e-16
- joint foot_3_to_calf_3: origin xyz=1.58779e-08 0.3 -5.96046e-08 rpy=2.35619 8.27288e-08 2.31242e-08 -> xyz=5.36083e-17 0.3 0 rpy=2.35619 6.80001e-18 3.69787e-17

Commit message: saving pose matching controller
but it is not what I expected. some seems wrong. it is not lifting the legs need to debug that.

File: newton-4.00/applications/media/quadSpider.urdf (robot description, URDF)
Before this commit: robot robot_model, 13 links, 12 joints
Joints:
- joint calf_0_to_thigh_0: limit lower=-1.047197 upper=1.047197 effort=1000.000000 velocity=0.500000 -> lower=-1.221730 upper=1.221730 effort=1000.000000 velocity=0.500000; origin xyz=0.3 -5.55112e-17 2.39534e-17 rpy=3.14159 1.5708 0 -> xyz=0.3 -5.96046e-08 8.45571e-09 rpy=3.14159 1.5708 0
- joint calf_1_to_thigh_1: limit lower=-1.047197 upper=1.047197 effort=1000.000000 velocity=0.500000 -> lower=-1.221730 upper=1.221730 effort=1000.000000 velocity=0.500000; origin xyz=0.3 1.11022e-16 5.07754e-17 rpy=3.14159 1.5708 0 -> xyz=0.3 8.9407e-08 1.6562e-08 rpy=3.14159 1.5708 0
- joint calf_2_to_thigh_2: limit lower=-1.047197 upper=1.047197 effort=1000.000000 velocity=0.500000 -> lower=-1.221730 upper=1.221730 effort=1000.000000 velocity=0.500000; origin xyz=0.3 2.77556e-17 2.45631e-17 rpy=-3.14159 -1.5708 0 -> xyz=0.3 -1.49012e-08 6.70279e-09 rpy=-3.14159 -1.5708 0
- joint calf_3_to_thigh_3: limit lower=-1.047197 upper=1.047197 effort=1000.000000 velocity=0.500000 -> lower=-1.221730 upper=1.221730 effort=1000.000000 velocity=0.500000; origin xyz=0.3 -2.77556e-17 -2.45058e-17 rpy=-3.14159 -1.5708 0 -> xyz=0.3 -2.98023e-08 -3.28874e-08 rpy=-3.14159 -1.5708 0
- joint foot_0_to_calf_0: origin xyz=3.08777e-17 0.3 -5.55112e-17 rpy=-0.785398 -4.88977e-17 -3.14159 -> xyz=-3.05751e-08 0.3 -2.98023e-08 rpy=-0.785398 5.76315e-08 3.14159
- joint foot_1_to_calf_1: origin xyz=-2.54984e-17 0.3 -5.55112e-17 rpy=-0.785398 4.80945e-17 3.14159 -> xyz=2.74028e-08 0.3 5.96046e-08 rpy=-0.785398 6.94903e-08 -3.14159
- joint foot_2_to_calf_2: origin xyz=-7.58832e-17 0.3 -5.55112e-17 rpy=2.35619 -4.40315e-17 -1.85238e-16 -> xyz=3.42348e-08 0.3 -2.98023e-08 rpy=2.35619 -2.52655e-08 8.44092e-08
- joint foot_3_to_calf_3: origin xyz=5.36083e-17 0.3 0 rpy=2.35619 6.80001e-18 3.69787e-17 -> xyz=7.59102e-09 0.3 -2.98023e-08 rpy=2.35619 9.57024e-09 -3.09262e-08
