Commit message: saving latest model.

File: newton-4.00/applications/media/cartpole.urdf (robot description, URDF)
Before this commit: robot physics, 1 links, 0 joints
Links:
- added link pole_link, mass 10.0; collision cylinder length=0.4 radius=0.05; visual cylinder length=0.4 radius=0.05
Joints:
- added joint pole_link_base_link: type continuous, parent base_link, child pole_link, origin xyz=0 0 0 rpy=0 0 0, axis 0 1 0

Commit message: enabling cartpole discrete using urdf file

File: newton-4.00/applications/media/cartpole.urdf (robot description, URDF)
Before this commit: robot physics, 2 links, 1 joints
Links:
- removed link pole_link
- added link node_0_link, mass 10; collision cylinder length=0.46 radius=0.03; visual cylinder length=0.46 radius=0.03
Joints:
- removed joint pole_link_base_link
- added joint node_0_link_to_base_link: type continuous, parent base_link, child node_0_link, origin xyz=0 0 0 rpy=6.27833e-07 1.5708 0, axis 3.13916e-07 1 -3.13916e-07

Commit message: added newton extension that allows cylinder, capsule and wheels.

File: newton-4.00/applications/media/cartpole.urdf (robot description, URDF)
Before this commit: robot robot_model, 2 links, 1 joints
Links:
- link node_0_link: geometry collision cylinder length=0.47 radius=0.035; visual cylinder length=0.47 radius=0.035
Joints:
- joint node_0_link_to_base_link: origin xyz=0 0 0 rpy=6.27833e-07 1.5708 0 -> xyz=0 9.8099e-09 0.03125 rpy=6.27833e-07 1.5708 0

Commit message: apply proper rotation to visual model.

File: newton-4.00/applications/media/cartpole.urdf (robot description, URDF)
Before this commit: robot robot_model, 2 links, 1 joints
Links:
- removed link node_0_link
- added link pole_link, mass 10; collision cylinder length=0.5 radius=0.05; visual cylinder length=0.5 radius=0.05
Joints:
- removed joint node_0_link_to_base_link
- added joint pole_link_to_base_link: type continuous, parent base_link, child pole_link, origin xyz=0 1.96198e-08 0.0625 rpy=3.13916e-07 -0 1.5708

Commit message: start adding continue Proxima policy trainer (wip)
start adding con

File: newton-4.00/applications/media/cartpole.urdf (robot description, URDF)
Before this commit: robot robot_model, 2 links, 1 joints
Joints:
- joint pole_link_to_base_link: origin xyz=0 1.96198e-08 0.0625 rpy=3.13916e-07 -0 1.5708 -> xyz=0 0.0 0.0625 rpy=0.0 0.0 1.5708
