Commit message: setting up quad 1 to use urdf file. (wip)

File: newton-4.00/applications/media/unicycle.urdf (robot description, URDF)
Before this commit: robot robot_model, 3 links, 2 joints
Joints:
- joint node_0_link_to_node_1_link: origin xyz=-4.52987e-08 -4.52987e-08 0.3 rpy=0 -0 -1.68775e-21 -> xyz=-9.41749e-08 -9.41749e-08 0.3 rpy=0 -0 0
- joint node_1_link_to_base_link: origin xyz=0 -3.01992e-08 -0.2 rpy=3.14159 -3.01992e-07 -1.5708 -> xyz=0 -6.27833e-08 -0.2 rpy=3.14159 -6.27833e-07 -1.5708

Commit message: removed all file format legacy

File: newton-4.00/applications/media/unicycle.urdf (robot description, URDF)
Before this commit: robot robot_model, 3 links, 2 joints
Links:
- removed link node_0_link
- removed link node_1_link
- added link leg, mass 1; collision cylinder length=0.35 radius=0.025; visual cylinder length=0.35 radius=0.025
- added link wheel, mass 1; collision sphere radius=0.1; visual sphere radius=0.1
Joints:
- removed joint node_0_link_to_node_1_link
- removed joint node_1_link_to_base_link
- added joint leg_to_base_link: type continuous, parent base_link, child leg, origin xyz=0 -6.27833e-08 -0.2 rpy=3.14159 -6.27833e-07 -1.5708
- added joint wheel_to_leg: type continuous, parent leg, child wheel, origin xyz=-9.41749e-08 -9.41749e-08 0.3 rpy=0 -0 0

Commit message: added some more tweaks
A more robust and stable controller.
Enhancements include:
Angular drag applied at the top box
Random lateral push
Lasso regularization replacing Ridge

These adjustments result in a significantly more stable controller,
capable of recovering from moderate disturbances.

File: newton-4.00/applications/media/unicycle.urdf (robot description, URDF)
Before this commit: robot robot_model, 3 links, 2 joints
Links:
- link base_link: geometry collision box size=0.703125 0.9375 0.585938; visual box size=0.703125 0.9375 0.585938
- link leg: geometry collision box size=0.1 0.1 0.1; visual box size=0.1 0.1 0.1
- link wheel: mass 1 -> 5; geometry collision sphere radius=0.3; visual sphere radius=0.3
Joints:
- joint leg_to_base_link: origin xyz=0 -6.27833e-08 -0.2 rpy=3.14159 -6.27833e-07 -1.5708 -> xyz=1.24939e-08 4.31586e-08 0.285827 rpy=-1.5708 -1.43052e-06 -1.5708
- joint wheel_to_leg: origin xyz=-9.41749e-08 -9.41749e-08 0.3 rpy=0 -0 0 -> xyz=-1.57073e-06 1.82075 -9.48105e-09 rpy=1.38046e-13 6.39126e-07 -3.14159
